File: Battery_protections.kicad_sch (KiCad schematic)
At the start: 27 parts, among them J6 thermistor, Q2 SI2102A-TP, Q3 SI2102A-TP, Q4 SI2102A-TP, Q5 SI2102A-TP, Q6 SI2102A-TP, U4 BQ29209DRBR, U5 AP9101CK6, U6 AP9101CK6, U7 LM358

Commit message: Fixes brought on laptop
Parts:
- removed R14: 10K, Resistor_SMD:R_0805_2012Metric_Pad1.20x1.40mm_HandSolder, symbol Device:R_US
Changed lines of the file:
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@@
   (junction (at 110.49 100.33) (diameter 0) (color 0 0 0 0)
   )
-  (junction (at 152.4 102.87) (diameter 0) (color 0 0 0 0)
-  )
   (junction (at 105.41 58.42) (diameter 0) (color 0 0 0 0)
   )
@@
   )
   (junction (at 62.23 161.29) (diameter 0) (color 0 0 0 0)
-  )
-  (junction (at 132.08 119.38) (diameter 0) (color 0 0 0 0)
   )
   (junction (at 105.41 78.74) (diameter 0) (color 0 0 0 0)
@@
     (stroke (width 0) (type default) (color 0 0 0 0))
   )
-  (wire (pts (xy 152.4 114.3) (xy 152.4 119.38))
-    (stroke (width 0) (type default) (color 0 0 0 0))
-  )
   (wire (pts (xy 143.51 36.83) (xy 156.21 36.83))
     (stroke (width 0) (type default) (color 0 0 0 0))
@@
     (stroke (width 0) (type default) (color 0 0 0 0))
   )
-  (wire (pts (xy 142.24 102.87) (xy 152.4 102.87))
+  (wire (pts (xy 142.24 102.87) (xy 157.48 102.87))
     (stroke (width 0) (type default) (color 0 0 0 0))
   )
@@
     (stroke (width 0) (type default) (color 0 0 0 0))
   )
-  (wire (pts (xy 165.1 118.11) (xy 181.61 118.11))
+  (wire (pts (xy 165.1 119.38) (xy 181.61 119.38))
     (stroke (width 0) (type default) (color 0 0 0 0))
   )
@@
     (stroke (width 0) (type default) (color 0 0 0 0))
   )
-  (wire (pts (xy 152.4 102.87) (xy 152.4 106.68))
-    (stroke (width 0) (type default) (color 0 0 0 0))
-  )
   (wire (pts (xy 62.23 161.29) (xy 62.23 162.56))
     (stroke (width 0) (type default) (color 0 0 0 0))
@@
     (stroke (width 0) (type default) (color 0 0 0 0))
   )
-  (wire (pts (xy 132.08 119.38) (xy 152.4 119.38))
-    (stroke (width 0) (type default) (color 0 0 0 0))
-  )
   (wire (pts (xy 158.75 173.99) (xy 158.75 177.8))
     (stroke (width 0) (type default) (color 0 0 0 0))
@@
     (stroke (width 0) (type default) (color 0 0 0 0))
   )
-  (wire (pts (xy 165.1 107.95) (xy 165.1 118.11))
+  (wire (pts (xy 165.1 107.95) (xy 165.1 119.38))
     (stroke (width 0) (type default) (color 0 0 0 0))
   )
@@
   )
   (wire (pts (xy 133.35 49.53) (xy 133.35 46.99))
-    (stroke (width 0) (type default) (color 0 0 0 0))
-  )
-  (wire (pts (xy 152.4 102.87) (xy 157.48 102.87))
     (stroke (width 0) (type default) (color 0 0 0 0))
   )
@@
     (effects (font (size 1.27 1.27)) (justify right bottom))
   )
-  (label "Batt -" (at 181.61 118.11 180)
+  (label "Batt -" (at 181.61 119.38 180)
     (effects (font (size 1.27 1.27)) (justify right bottom))
   )
@@
       (effects (font (size 1.27 1.27)) hide)
     )
-    (pin "1")
-    (pin "2")
-  )
-  (symbol (lib_id "Device:R_US") (at 152.4 110.49 0) (unit 1)
-    (in_bom yes) (on_board yes)
-    (property "Reference" "R14" (id 0) (at 151.13 115.57 90))
-    (property "Value" "10K" (id 1) (at 151.13 105.41 90))
-    (property "Footprint" "Resistor_SMD:R_0805_2012Metric_Pad1.20x1.40mm_HandSolder" (id 2) (at 153.416 110.744 90)
-      (effects (font (size 1.27 1.27)) hide)
-    )
-    (property "Datasheet" "https://www.seielect.com/catalog/sei-rncp.pdf" (id 3) (at 152.4 110.49 0)
-      (effects (font (size 1.27 1.27)) hide)
-    )
-    (property "Digikey link" "https://www.digikey.ca/en/products/detail/stackpole-electronics-inc/RNCP0805FTD10K0/2240262" (id 4) (at 152.4 110.49 90)
-      (effects (font (size 1.27 1.27)) hide)
-    )
-    (property "Part number" "RNCP0805FTD10K0" (id 5) (at 152.4 110.49 90)
-      (effects (font (size 1.27 1.27)) hide)
-    )

Commit message: Initial layout
Parts:
- removed R13: 100, Resistor_SMD:R_0805_2012Metric_Pad1.20x1.40mm_HandSolder, symbol Device:R_US
- added R?: 100, Resistor_SMD:R_0805_2012Metric_Pad1.20x1.40mm_HandSolder, symbol Device:R_US
Connections:
- net CO_1: no longer Q4.1 (G), U6.3 (CO)
- net DO_1: no longer Q5.1 (G), U6.1 (DO)
- net SW_Batt +: now also R?.2; no longer C13.1
- net at U4.7 (VDD): now also C13.1, R?.1
- new net CO_2: Q4.1 (G), U6.3 (CO)
- new net DO_2: Q5.1 (G), U6.1 (DO)
Other:
- moved on the sheet: C13
Changed lines of the file:
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@@
   (junction (at 62.23 162.56) (diameter 0) (color 0 0 0 0)
   )
-  (junction (at 158.75 163.83) (diameter 0) (color 0 0 0 0)
-  )
   (junction (at 110.49 119.38) (diameter 0) (color 0 0 0 0)
   )
@@
   )
   (junction (at 105.41 78.74) (diameter 0) (color 0 0 0 0)
+  )
+  (junction (at 148.59 163.83) (diameter 0) (color 0 0 0 0)
   )
   (junction (at 105.41 49.53) (diameter 0) (color 0 0 0 0)
@@
     (stroke (width 0) (type default) (color 0 0 0 0))
   )
-  (wire (pts (xy 158.75 163.83) (xy 170.18 163.83))
-    (stroke (width 0) (type default) (color 0 0 0 0))
-  )
   (wire (pts (xy 165.1 24.13) (xy 177.8 24.13))
     (stroke (width 0) (type default) (color 0 0 0 0))
@@
     (stroke (width 0) (type default) (color 0 0 0 0))
   )
+  (wire (pts (xy 148.59 148.59) (xy 148.59 152.4))
+    (stroke (width 0) (type default) (color 0 0 0 0))
+  )
   (wire (pts (xy 110.49 100.33) (xy 127 100.33))
     (stroke (width 0) (type default) (color 0 0 0 0))
@@
     (stroke (width 0) (type default) (color 0 0 0 0))
   )
-  (wire (pts (xy 151.13 163.83) (xy 158.75 163.83))
-    (stroke (width 0) (type default) (color 0 0 0 0))
-  )
   (wire (pts (xy 85.09 119.38) (xy 110.49 119.38))
     (stroke (width 0) (type default) (color 0 0 0 0))
@@
     (stroke (width 0) (type default) (color 0 0 0 0))
   )
+  (wire (pts (xy 163.83 148.59) (xy 148.59 148.59))
+    (stroke (width 0) (type default) (color 0 0 0 0))
+  )
   (wire (pts (xy 105.41 58.42) (xy 105.41 63.5))
     (stroke (width 0) (type default) (color 0 0 0 0))
@@
     (stroke (width 0) (type default) (color 0 0 0 0))
   )
+  (wire (pts (xy 148.59 163.83) (xy 148.59 166.37))
+    (stroke (width 0) (type default) (color 0 0 0 0))
+  )
   (wire (pts (xy 165.1 38.1) (xy 165.1 40.64))
     (stroke (width 0) (type default) (color 0 0 0 0))
@@
     (stroke (width 0) (type default) (color 0 0 0 0))
   )
-  (wire (pts (xy 158.75 173.99) (xy 158.75 177.8))
+  (wire (pts (xy 148.59 173.99) (xy 148.59 177.8))
     (stroke (width 0) (type default) (color 0 0 0 0))
   )
@@
     (stroke (width 0) (type default) (color 0 0 0 0))
   )
-  (wire (pts (xy 128.27 163.83) (xy 143.51 163.83))
+  (wire (pts (xy 148.59 160.02) (xy 148.59 163.83))
     (stroke (width 0) (type default) (color 0 0 0 0))
   )
@@
     (stroke (width 0) (type default) (color 0 0 0 0))
   )
-  (wire (pts (xy 158.75 163.83) (xy 158.75 166.37))
-    (stroke (width 0) (type default) (color 0 0 0 0))
-  )
   (wire (pts (xy 165.1 80.01) (xy 165.1 97.79))
     (stroke (width 0) (type default) (color 0 0 0 0))
@@
     (stroke (width 0) (type default) (color 0 0 0 0))
   )
+  (wire (pts (xy 128.27 163.83) (xy 148.59 163.83))
+    (stroke (width 0) (type default) (color 0 0 0 0))
+  )
   (wire (pts (xy 133.35 49.53) (xy 133.35 46.99))
     (stroke (width 0) (type default) (color 0 0 0 0))
@@
     (effects (font (size 1.27 1.27)) (justify left bottom))
   )
-  (label "DO_1" (at 148.59 71.12 0)
+  (label "DO_2" (at 148.59 71.12 0)
     (effects (font (size 1.27 1.27)) (justify left bottom))
   )
@@
     (effects (font (size 1.27 1.27)) (justify left bottom))
   )
-  (label "CO_1" (at 148.59 66.04 0)
+  (label "CO_2" (at 148.59 66.04 0)
     (effects (font (size 1.27 1.27)) (justify left bottom))
   )
@@
     (effects (font (size 1.27 1.27)) (justify left bottom))
   )
-  (label "SW_Batt +" (at 170.18 163.83 180)
+  (label "SW_Batt +" (at 163.83 148.59 180)
     (effects (font (size 1.27 1.27)) (justify right bottom))
   )
@@
     (pin "2")
   )
-  (symbol (lib_id "power:GND") (at 158.75 177.8 0) (unit 1)
-    (in_bom yes) (on_board yes) (fields_autoplaced)
-    (property "Reference" "#PWR016" (id 0) (at 158.75 184.15 0)
-      (effects (font (size 1.27 1.27)) hide)
-    )
-    (property "Value" "GND" (id 1) (at 158.75 182.88 0))
-    (property "Footprint" "" (id 2) (at 158.75 177.8 0)
-      (effects (font (size 1.27 1.27)) hide)
-    )
-    (property "Datasheet" "" (id 3) (at 158.75 177.8 0)
+  (symbol (lib_id "power:GND") (at 148.59 177.8 0) (unit 1)
+    (in_bom yes) (on_board yes) (fields_autoplaced)
+    (property "Reference" "#PWR016" (id 0) (at 148.59 184.15 0)
+      (effects (font (size 1.27 1.27)) hide)
+    )
+    (property "Value" "GND" (id 1) (at 148.59 182.88 0))
+    (property "Footprint" "" (id 2) (at 148.59 177.8 0)
+      (effects (font (size 1.27 1.27)) hide)
+    )
+    (property "Datasheet" "" (id 3) (at 148.59 177.8 0)
       (effects (font (size 1.27 1.27)) hide)
     )
@@
     (pin "6")
   )
+  (symbol (lib_id "Device:R_US") (at 148.59 156.21 180) (unit 1)
+    (in_bom yes) (on_board yes)
+    (property "Reference" "R?" (id 0) (at 149.86 152.4 90))
+    (property "Value" "100" (id 1) (at 149.86 160.02 90))
+    (property "Footprint" "Resistor_SMD:R_0805_2012Metric_Pad1.20x1.40mm_HandSolder" (id 2) (at 147.574 155.956 90)
+      (effects (font (size 1.27 1.27)) hide)
+    )
+    (property "Datasheet" "https://www.seielect.com/catalog/sei-rmcf_rmcp.pdf" (id 3) (at 148.59 156.21 0)
+      (effects (font (size 1.27 1.27)) hide)
+    )
+    (property "Digikey link" "https://www.digikey.ca/en/products/detail/stackpole-electronics-inc/RMCF0805FT100R/1760711" (id 4) (at 148.59 156.21 90)
+      (effects (font (size 1.27 1.27)) hide)
+    )
+    (property "Part number" "RMCF0805FT100R" (id 5) (at 148.59 156.21 90)
+      (effects (font (size 1.27 1.27)) hide)
+    )
+    (pin "1")
+    (pin "2")
+  )
   (symbol (lib_id "Device:R_US") (at 53.34 162.56 270) (unit 1)
     (in_bom yes) (on_board yes)
@@
     (pin "2")
   )
-  (symbol (lib_id "Device:C") (at 158.75 170.18 0) (unit 1)
-    (in_bom yes) (on_board yes) (fields_autoplaced)
-    (property "Reference" "C13" (id 0) (at 162.56 168.9099 0)
-      (effects (font (size 1.27 1.27)) (justify left))
-    )
-    (property "Value" "100nF" (id 1) (at 162.56 171.4499 0)
-      (effects (font (size 1.27 1.27)) (justify left))
-    )
-    (property "Footprint" "Capacitor_SMD:C_0805_2012Metric_Pad1.18x1.45mm_HandSolder" (id 2) (at 159.7152 173.99 0)
-      (effects (font (size 1.27 1.27)) hide)
-    )
-    (property "Datasheet" "https://www.seielect.com/Catalog/SEI-CML.PDF" (id 3) (at 158.75 170.18 0)
-      (effects (font (size 1.27 1.27)) hide)
-    )
-    (property "Digikey link" "https://www.digikey.ca/en/products/detail/stackpole-electronics-inc/CML0805Y5V104ZT50V/10660028" (id 4) (at 158.75 170.18 0)
-      (effects (font (size 1.27 1.27)) hide)
-    )
-    (property "Part number" "CML0805Y5V104ZT50V" (id 5) (at 158.75 170.18 0)
+  (symbol (lib_id "Device:C") (at 148.59 170.18 0) (unit 1)
+    (in_bom yes) (on_board yes) (fields_autoplaced)
+    (property "Reference" "C13" (id 0) (at 152.4 168.9099 0)
+      (effects (font (size 1.27 1.27)) (justify left))
+    )
+    (property "Value" "100nF" (id 1) (at 152.4 171.4499 0)
+      (effects (font (size 1.27 1.27)) (justify left))
+    )
+    (property "Footprint" "Capacitor_SMD:C_0805_2012Metric_Pad1.18x1.45mm_HandSolder" (id 2) (at 149.5552 173.99 0)
+      (effects (font (size 1.27 1.27)) hide)
+    )
+    (property "Datasheet" "https://www.seielect.com/Catalog/SEI-CML.PDF" (id 3) (at 148.59 170.18 0)
+      (effects (font (size 1.27 1.27)) hide)
+    )
+    (property "Digikey link" "https://www.digikey.ca/en/products/detail/stackpole-electronics-inc/CML0805Y5V104ZT50V/10660028" (id 4) (at 148.59 170.18 0)
+      (effects (font (size 1.27 1.27)) hide)
+    )
+    (property "Part number" "CML0805Y5V104ZT50V" (id 5) (at 148.59 170.18 0)
       (effects (font (size 1.27 1.27)) hide)
     )
@@
     (pin "1")
   )
-  (symbol (lib_id "Device:R_US") (at 147.32 163.83 90) (unit 1)
-    (in_bom yes) (on_board yes)
-    (property "Reference" "R13" (id 0) (at 151.13 165.1 90))
-    (property "Value" "100" (id 1) (at 143.51 165.1 90))
-    (property "Footprint" "Resistor_SMD:R_0805_2012Metric_Pad1.20x1.40mm_HandSolder" (id 2) (at 147.574 162.814 90)
-      (effects (font (size 1.27 1.27)) hide)
-    )
-    (property "Datasheet" "https://www.seielect.com/catalog/sei-rmcf_rmcp.pdf" (id 3) (at 147.32 163.83 0)
-      (effects (font (size 1.27 1.27)) hide)
-    )
-    (property "Digikey link" "https://www.digikey.ca/en/products/detail/stackpole-electronics-inc/RMCF0805FT100R/1760711" (id 4) (at 147.32 163.83 90)
-      (effects (font (size 1.27 1.27)) hide)
-    )
-    (property "Part number" "RMCF0805FT100R" (id 5) (at 147.32 163.83 90)
-      (effects (font (size 1.27 1.27)) hide)
-    )
-    (pin "1")
-    (pin "2")
-  )
   (symbol (lib_id "power:GND") (at 111.76 184.15 0) (unit 1)

Commit message: Last commit from desktop
Parts:
- gave numbers to parts that had none: 1
Changed lines of the file:
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@@
   (symbol (lib_id "Device:R_US") (at 148.59 156.21 180) (unit 1)
     (in_bom yes) (on_board yes)
-    (property "Reference" "R?" (id 0) (at 149.86 152.4 90))
+    (property "Reference" "R13" (id 0) (at 149.86 152.4 90))
     (property "Value" "100" (id 1) (at 149.86 160.02 90))
     (property "Footprint" "Resistor_SMD:R_0805_2012Metric_Pad1.20x1.40mm_HandSolder" (id 2) (at 147.574 155.956 90)

Commit message: First layout done
Connections:
- net CB_EN is gone; now on net GND: U4.6 (*CB_EN)
- net SW_Batt +: no longer R5.2
- net batt -: no longer R7.2
- new net Bal_batt_+: R5.2
- new net Bal_batt_-: R7.2
Changed lines of the file:
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@@
   (junction (at 62.23 147.32) (diameter 0) (color 0 0 0 0)
+  )
+  (junction (at 133.35 168.91) (diameter 0) (color 0 0 0 0)
   )
   (junction (at 120.65 119.38) (diameter 0) (color 0 0 0 0)
@@
     (stroke (width 0) (type default) (color 0 0 0 0))
   )
-  (wire (pts (xy 128.27 166.37) (xy 132.08 166.37))
+  (wire (pts (xy 128.27 166.37) (xy 133.35 166.37))
     (stroke (width 0) (type default) (color 0 0 0 0))
   )
@@
     (stroke (width 0) (type default) (color 0 0 0 0))
   )
+  (wire (pts (xy 133.35 166.37) (xy 133.35 168.91))
+    (stroke (width 0) (type default) (color 0 0 0 0))
+  )
   (wire (pts (xy 165.1 119.38) (xy 181.61 119.38))
     (stroke (width 0) (type default) (color 0 0 0 0))
@@
     (effects (font (size 1.27 1.27)) (justify left bottom))
   )
-  (label "Batt -" (at 38.1 175.26 0)
+  (label "Bal_batt_-" (at 38.1 175.26 0)
     (effects (font (size 1.27 1.27)) (justify left bottom))
   )
@@
     (effects (font (size 1.27 1.27)) (justify left bottom))
   )
-  (label "SW_Batt +" (at 38.1 147.32 0)
+  (label "Bal_bat_+" (at 38.1 147.32 0)
     (effects (font (size 1.27 1.27)) (justify left bottom))
   )
@@
     (effects (font (size 1.27 1.27)) (justify right bottom))
   )
+  (hierarchical_label "batt -" (shape input) (at 181.61 119.38 0)
+    (effects (font (size 1.27 1.27)) (justify left))
+  )
+  (hierarchical_label "Bal_batt_+" (shape input) (at 31.75 160.02 180)
+    (effects (font (size 1.27 1.27)) (justify right))
+  )
+  (hierarchical_label "Bal_batt_-" (shape input) (at 31.75 165.1 180)
+    (effects (font (size 1.27 1.27)) (justify right))
+  )
   (hierarchical_label "Batt mid" (shape input) (at 31.75 162.56 180)
-    (effects (font (size 1.27 1.27)) (justify right))
-  )
-  (hierarchical_label "batt -" (shape input) (at 31.75 165.1 180)
     (effects (font (size 1.27 1.27)) (justify right))
   )
@@
     (effects (font (size 1.27 1.27)) (justify right))
   )
-  (hierarchical_label "SW_Batt +" (shape input) (at 31.75 160.02 180)
-    (effects (font (size 1.27 1.27)) (justify right))
-  )
-  (hierarchical_label "CB_EN" (shape input) (at 132.08 166.37 0)
-    (effects (font (size 1.27 1.27)) (justify left))
+  (hierarchical_label "SW_Batt +" (shape input) (at 80.01 29.21 180)
+    (effects (font (size 1.27 1.27)) (justify right))
   )
   (symbol (lib_id "Battery_Management:AP9101CK6") (at 133.35 68.58 0) (unit 1)
