File: Charging.kicad_sch (KiCad schematic)
At the start: 7 parts, among them Q1 SI2301-TP, U3 MCP73844T-820I/MS

Commit message: 1st Gerber creatd  Please enter the commit message for your changes. Lines starting
Parts:
- removed Q1: SI2301-TP, Package_TO_SOT_SMD:SOT-323_SC-70, symbol Transistor_FET:SI2301-TP
- added C8: 10uF, Capacitor_SMD:C_0805_2012Metric_Pad1.18x1.45mm_HandSolder, symbol Device:C_Polarized_Small_US
- added Q1: IRF7404, Package_SO:SOIC-8_3.9x4.9mm_P1.27mm, symbol Transistor_FET:IRF7404
- renumbered D5 to D3
Connections:
- net CHG_OUT +: now also C8.1, Q1.5 (D), Q1.6 (D), Q1.7 (D), Q1.8 (D)
- net GND: now also C8.2
- net at R4.1, U3.1 (SENSE): now also Q1.1 (S), Q1.2 (S), Q1.3 (S)
- net at U3.8 (DRV): now also Q1.4 (G)
Changed lines of the file:
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@@
   (junction (at 123.19 87.63) (diameter 0) (color 0 0 0 0)
   )
+  (junction (at 195.58 87.63) (diameter 0) (color 0 0 0 0)
+  )
   (junction (at 118.11 87.63) (diameter 0) (color 0 0 0 0)
   )
-  (junction (at 195.58 87.63) (diameter 0) (color 0 0 0 0)
+  (junction (at 137.16 87.63) (diameter 0) (color 0 0 0 0)
+  )
+  (junction (at 208.28 87.63) (diameter 0) (color 0 0 0 0)
   )
   (junction (at 106.68 87.63) (diameter 0) (color 0 0 0 0)
   )
-  (junction (at 137.16 87.63) (diameter 0) (color 0 0 0 0)
-  )
-  (wire (pts (xy 195.58 87.63) (xy 215.9 87.63))
+  (wire (pts (xy 195.58 87.63) (xy 208.28 87.63))
     (stroke (width 0) (type default) (color 0 0 0 0))
   )
@@
     (stroke (width 0) (type default) (color 0 0 0 0))
   )
+  (wire (pts (xy 208.28 97.79) (xy 208.28 101.6))
+    (stroke (width 0) (type default) (color 0 0 0 0))
+  )
   (wire (pts (xy 140.97 100.33) (xy 137.16 100.33))
     (stroke (width 0) (type default) (color 0 0 0 0))
   )
+  (wire (pts (xy 208.28 87.63) (xy 208.28 92.71))
+    (stroke (width 0) (type default) (color 0 0 0 0))
+  )
   (wire (pts (xy 153.67 91.44) (xy 153.67 92.71))
     (stroke (width 0) (type default) (color 0 0 0 0))
@@
     (stroke (width 0) (type default) (color 0 0 0 0))
   )
+  (wire (pts (xy 187.96 95.25) (xy 187.96 100.33))
+    (stroke (width 0) (type default) (color 0 0 0 0))
+  )
   (wire (pts (xy 153.67 118.11) (xy 153.67 119.38))
     (stroke (width 0) (type default) (color 0 0 0 0))
   )
-  (wire (pts (xy 187.96 100.33) (xy 187.96 95.25))
-    (stroke (width 0) (type default) (color 0 0 0 0))
-  )
   (wire (pts (xy 177.8 119.38) (xy 177.8 121.92))
     (stroke (width 0) (type default) (color 0 0 0 0))
@@
   )
   (wire (pts (xy 140.97 107.95) (xy 118.11 107.95))
+    (stroke (width 0) (type default) (color 0 0 0 0))
+  )
+  (wire (pts (xy 208.28 87.63) (xy 215.9 87.63))
     (stroke (width 0) (type default) (color 0 0 0 0))
   )
@@
     (pin "8")
   )
-  (symbol (lib_id "Transistor_FET:SI2301-TP") (at 187.96 90.17 270) (mirror x) (unit 1)
-    (in_bom yes) (on_board yes)
-    (property "Reference" "Q1" (id 0) (at 187.96 81.28 90))
-    (property "Value" "SI2301-TP" (id 1) (at 187.96 83.82 90))
-    (property "Footprint" "Package_TO_SOT_SMD:SOT-323_SC-70" (id 2) (at 170.18 99.06 0)
+  (symbol (lib_id "Transistor_FET:IRF7404") (at 187.96 90.17 270) (mirror x) (unit 1)
+    (in_bom yes) (on_board yes) (fields_autoplaced)
+    (property "Reference" "Q1" (id 0) (at 187.96 80.01 90))
+    (property "Value" "IRF7404" (id 1) (at 187.96 82.55 90))
+    (property "Footprint" "Package_SO:SOIC-8_3.9x4.9mm_P1.27mm" (id 2) (at 186.055 85.09 0)
       (effects (font (size 1.27 1.27) italic) (justify left) hide)
     )
-    (property "Datasheet" "https://www.mccsemi.com/pdf/Products/SI2301(SOT-23).pdf" (id 3) (at 166.37 109.22 0)
+    (property "Datasheet" "http://www.infineon.com/dgdl/irf7404.pdf?fileId=5546d462533600a4015355fa2b5b1b9e" (id 3) (at 187.96 90.17 90)
       (effects (font (size 1.27 1.27)) (justify left) hide)
     )
-    (property "Digikey link" "https://www.digikey.ca/en/products/detail/micro-commercial-co/SI2301-TP/1793242" (id 4) (at 162.56 81.28 0)
-      (effects (font (size 1.27 1.27)) hide)
-    )
-    (property "Part number" "SI2301-TP" (id 5) (at 173.99 87.63 0)
-      (effects (font (size 1.27 1.27)) hide)
-    )
     (pin "1")
     (pin "2")
     (pin "3")
+    (pin "4")
+    (pin "5")
+    (pin "6")
+    (pin "7")
+    (pin "8")
+  )
+  (symbol (lib_id "power:GND") (at 208.28 101.6 0) (mirror y) (unit 1)
+    (in_bom yes) (on_board yes) (fields_autoplaced)
+    (property "Reference" "#PWR013" (id 0) (at 208.28 107.95 0)
+      (effects (font (size 1.27 1.27)) hide)
+    )
+    (property "Value" "GND" (id 1) (at 210.82 102.8699 0)
+      (effects (font (size 1.27 1.27)) (justify right))
+    )
+    (property "Footprint" "" (id 2) (at 208.28 101.6 0)
+      (effects (font (size 1.27 1.27)) hide)
+    )
+    (property "Datasheet" "" (id 3) (at 208.28 101.6 0)
+      (effects (font (size 1.27 1.27)) hide)
+    )
+    (pin "1")
   )
   (symbol (lib_id "Device:R_US") (at 129.54 87.63 270) (unit 1)
@@
   (symbol (lib_id "LED:CQY99") (at 129.54 104.14 180) (unit 1)
     (in_bom yes) (on_board yes)
-    (property "Reference" "D5" (id 0) (at 130.81 101.6 0))
+    (property "Reference" "D3" (id 0) (at 130.81 101.6 0))
     (property "Value" "Yellow" (id 1) (at 130.81 99.06 0))
     (property "Footprint" "LED_THT:LED_D3.0mm" (id 2) (at 129.54 108.585 0)
@@
       (effects (font (size 1.27 1.27)) hide)
     )
+    (pin "1")
+    (pin "2")
+  )
+  (symbol (lib_id "Device:C_Polarized_Small_US") (at 208.28 95.25 0) (unit 1)
+    (in_bom yes) (on_board yes) (fields_autoplaced)
+    (property "Reference" "C8" (id 0) (at 210.82 93.5481 0)
+      (effects (font (size 1.27 1.27)) (justify left))
+    )
+    (property "Value" "10uF" (id 1) (at 210.82 96.0881 0)
+      (effects (font (size 1.27 1.27)) (justify left))
+    )
+    (property "Footprint" "Capacitor_SMD:C_0805_2012Metric_Pad1.18x1.45mm_HandSolder" (id 2) (at 208.28 95.25 0)
+      (effects (font (size 1.27 1.27)) hide)
+    )
+    (property "Datasheet" "https://search.murata.co.jp/Ceramy/image/img/A01X/G101/ENG/GRM21BR61H106KE43-01A.pdf" (id 3) (at 208.28 95.25 0)
+      (effects (font (size 1.27 1.27)) hide)
+    )
+    (property "Digikey link" "https://www.digikey.ca/en/products/detail/murata-electronics/GRM21BR61H106KE43K/15191954" (id 4) (at 208.28 95.25 0)
+      (effects (font (size 1.27 1.27)) hide)
+    )
+    (property "Part number" "GRM21BR61H106KE43K" (id 5) (at 208.28 95.25 0)
+      (effects (font (size 1.27 1.27)) hide)
+    )
