File: Ki_PCB.kicad_pcb (KiCad board)
At the start: 2 copper layers, 0 parts

Commit message: Initial layout
Parts:
- added C1: 1uF, Capacitor_SMD:C_0805_2012Metric_Pad1.18x1.45mm_HandSolder, F.Cu at (76.3, 119.5)
- added C10: 330nF, Capacitor_SMD:C_0805_2012Metric_Pad1.18x1.45mm_HandSolder, F.Cu at (83.0, 108.0)
- added C11: 100nF, Capacitor_SMD:C_0805_2012Metric_Pad1.18x1.45mm_HandSolder, F.Cu at (111.1, 92.8)
- added C12: 100nF, Capacitor_SMD:C_0805_2012Metric_Pad1.18x1.45mm_HandSolder, F.Cu at (106.0, 92.8)
- added C13: 100nF, Capacitor_SMD:C_0805_2012Metric_Pad1.18x1.45mm_HandSolder, F.Cu at (78.2, 102.5)
- added C14: 100nF, Capacitor_SMD:C_0805_2012Metric_Pad1.18x1.45mm_HandSolder, F.Cu at (113.7, 105.4)
- added C15: 100nF, Capacitor_SMD:C_0805_2012Metric_Pad1.18x1.45mm_HandSolder, F.Cu at (125.5, 107.3)
- added C16: 1uF, Capacitor_SMD:C_0805_2012Metric_Pad1.18x1.45mm_HandSolder, F.Cu at (120.8, 112.3)
- added C17: 15nF, Capacitor_SMD:C_0805_2012Metric_Pad1.18x1.45mm_HandSolder, F.Cu at (112.5, 113.0)
- added C18: 120pF, Capacitor_SMD:C_0805_2012Metric_Pad1.18x1.45mm_HandSolder, F.Cu at (113.7, 109.8)
- added C19: 10nF, Capacitor_SMD:C_0805_2012Metric_Pad1.18x1.45mm_HandSolder, F.Cu at (124.5, 113.6)
- added C2: 4.7uF, Capacitor_SMD:C_0805_2012Metric_Pad1.18x1.45mm_HandSolder, F.Cu at (76.3, 124.8)
- added C20: 180uF, Capacitor_THT:CP_Radial_D8.0mm_P3.50mm, F.Cu at (127.1, 97.4)
- added C3: 1nF, Capacitor_SMD:C_0805_2012Metric_Pad1.18x1.45mm_HandSolder, F.Cu at (111.1, 132.2)
- added C4: 100nF, Capacitor_SMD:C_0805_2012Metric_Pad1.18x1.45mm_HandSolder, F.Cu at (116.4, 129.4)
- added C5: 100nF, Capacitor_SMD:C_0805_2012Metric_Pad1.18x1.45mm_HandSolder, F.Cu at (122.0, 135.5)
- added C6: 10uF, Capacitor_SMD:C_0805_2012Metric_Pad1.18x1.45mm_HandSolder, F.Cu at (86.3, 91.3)
- added C7: 100nF, Capacitor_SMD:C_0805_2012Metric_Pad1.18x1.45mm_HandSolder, F.Cu at (77.4, 96.1)
- added C8: 100nF, Capacitor_SMD:C_0805_2012Metric_Pad1.18x1.45mm_HandSolder, F.Cu at (77.4, 110.6)
- added C9: 100nF, Capacitor_SMD:C_0805_2012Metric_Pad1.18x1.45mm_HandSolder, F.Cu at (81.2, 110.6)
- added D1: Green, LED_THT:LED_D3.0mm, F.Cu at (132.1, 90.8)
- added D5: Yellow, LED_THT:LED_D3.0mm, F.Cu at (82.5, 91.3)
- added D6: CRS05(TE85L,Q,M), Diode_SMD:CRS05(TE85L,Q,M), F.Cu at (125.6, 92.0)
- added J1: 0039301020, Connector_Molex:Molex_Mini-Fit_Jr_5569-02A2_2x01_P4.20mm_Horizontal, F.Cu at (127.5, 82.8)
- added J2: B3B-XH-AM(LF)(SN), Connector_JST:JST_EH_B3B-EH-A_1x03_P2.50mm_Vertical, F.Cu at (133.7, 117.5)
- added J3: 0039301020, Connector_Molex:Molex_Mini-Fit_Jr_5569-02A2_2x01_P4.20mm_Horizontal, F.Cu at (82.1, 83.1)
- added J4: 0470531000, Connector:FanPinHeader_1x04_P2.54mm_Vertical, F.Cu at (133.7, 104.7)
- added J5: 4pin JST, Connector_JST:JST_EH_B4B-EH-A_1x04_P2.50mm_Vertical, F.Cu at (126.5, 83.4)
- added J6: thermistor, Connector_JST:JST_EH_B2B-EH-A_1x02_P2.50mm_Vertical, F.Cu at (129.6, 132.7)
- added L1: 100uH, Inductor_SMD:74404063101, F.Cu at (119.2, 92.0)
- added Q1: SI2301-TP, Package_TO_SOT_SMD:SOT-323_SC-70, F.Cu at (82.2, 100.2)
- added Q2: SI2102A-TP, Package_TO_SOT_SMD:SOT-323_SC-70, F.Cu at (112.6, 80.6)
- added Q3: SI2102A-TP, Package_TO_SOT_SMD:SOT-323_SC-70, F.Cu at (109.3, 80.6)
- added Q4: SI2102A-TP, Package_TO_SOT_SMD:SOT-323_SC-70, F.Cu at (106.5, 80.6)
- added Q5: SI2102A-TP, Package_TO_SOT_SMD:SOT-323_SC-70, F.Cu at (103.4, 80.6)
- added Q6: SI2102A-TP, Package_TO_SOT_SMD:SOT-323_SC-70, F.Cu at (100.4, 80.6)
- added Q7: SI2102A-TP, Package_TO_SOT_SMD:SOT-323_SC-70, F.Cu at (117.5, 102.8)
- added Q8: SI2102A-TP, Package_TO_SOT_SMD:SOT-323_SC-70, F.Cu at (118.8, 98.4)
- added R1: 510, Resistor_SMD:R_0805_2012Metric_Pad1.20x1.40mm_HandSolder, F.Cu at (128.7, 91.8)
- added R10: 22K, Resistor_SMD:R_0805_2012Metric_Pad1.20x1.40mm_HandSolder, F.Cu at (101.9, 98.1)
- added R11: 2K7, Resistor_SMD:R_0805_2012Metric_Pad1.20x1.40mm_HandSolder, F.Cu at (111.1, 85.7)
- added R12: 2K7, Resistor_SMD:R_0805_2012Metric_Pad1.20x1.40mm_HandSolder, F.Cu at (106.0, 85.7)
- added R13: 100, Resistor_SMD:R_0805_2012Metric_Pad1.20x1.40mm_HandSolder, F.Cu at (75.9, 102.5)
- added R15: 113K, Resistor_SMD:R_0805_2012Metric_Pad1.20x1.40mm_HandSolder, F.Cu at (125.5, 109.6)
- added R16: 100K, Resistor_SMD:R_0805_2012Metric_Pad1.20x1.40mm_HandSolder, F.Cu at (125.5, 105.0)
- added R17: 12K, Resistor_SMD:R_0805_2012Metric_Pad1.20x1.40mm_HandSolder, F.Cu at (111.2, 109.8)
- added R18: 10K, Resistor_SMD:R_0805_2012Metric_Pad1.20x1.40mm_HandSolder, F.Cu at (116.3, 98.4)
- added R19: 10K, Resistor_SMD:R_0805_2012Metric_Pad1.20x1.40mm_HandSolder, F.Cu at (120.1, 102.7)
- added R2: 22K, Resistor_SMD:R_0805_2012Metric_Pad1.20x1.40mm_HandSolder, F.Cu at (116.1, 137.5)
- added R20: 27K, Resistor_SMD:R_0805_2012Metric_Pad1.20x1.40mm_HandSolder, F.Cu at (127.7, 114.9)
- added R21: 2K7, Resistor_SMD:R_0805_2012Metric_Pad1.20x1.40mm_HandSolder, F.Cu at (116.9, 113.0)
- added R22: 200R, Resistor_SMD:R_0805_2012Metric_Pad1.20x1.40mm_HandSolder, F.Cu at (127.7, 112.3)
- added R3: 10K, Resistor_SMD:R_0805_2012Metric_Pad1.20x1.40mm_HandSolder, F.Cu at (86.3, 93.6)
- added R4: 0R110, Resistor_SMD:R_0805_2012Metric_Pad1.20x1.40mm_HandSolder, F.Cu at (87.3, 97.7)
- added R5: 261, Resistor_SMD:R_0805_2012Metric_Pad1.20x1.40mm_HandSolder, F.Cu at (76.7, 113.9)
- added R6: 261, Resistor_SMD:R_0805_2012Metric_Pad1.20x1.40mm_HandSolder, F.Cu at (79.2, 113.9)
- added R7: 442, Resistor_SMD:R_0805_2012Metric_Pad1.20x1.40mm_HandSolder, F.Cu at (81.7, 113.9)
- added R8: 330, Resistor_SMD:R_0805_2012Metric_Pad1.20x1.40mm_HandSolder, F.Cu at (111.0, 95.3)
- added R9: 330, Resistor_SMD:R_0805_2012Metric_Pad1.20x1.40mm_HandSolder, F.Cu at (106.0, 95.3)
- added RV1: 22K, Potentiometer_THT:PC16SH-10IP06-223A2020-TA, F.Cu at (96.7, 140.1)
- added RV2: 22K, Potentiometer_THT:3362P-1-223LF, F.Cu at (96.3, 100.4)
- added RV3: 5K, Potentiometer_THT:CT6EP502, F.Cu at (120.1, 118.1)
- added U1: LDL1117S50R, Package_TO_SOT_SMD:SOT-223-3_TabPin2, F.Cu at (81.3, 122.5)
- added U2: TLC555CPWR, Package_SO:TSSOP-14_4.4x5mm_P0.65mm, F.Cu at (116.4, 133.4)
- added U3: MCP73844T-820I/MS, Package_SO:MSOP-8_3x3mm_P0.65mm, F.Cu at (82.2, 96.9)
- added U4: BQ29209DRBR, My_footprints:BQ29209DRBR, F.Cu at (78.9, 107.0)
- added U5: AP9101CK6, Package_TO_SOT_SMD:SOT-23-6, F.Cu at (111.1, 89.4)
- added U6: AP9101CK6, Package_TO_SOT_SMD:SOT-23-6, F.Cu at (106.0, 89.2)
- added U7: LM358, Package_DIP:DIP-8_W7.62mm_LongPads, F.Cu at (93.8, 94.1)
- added U8: TL5001CDR, Package_SO:SOIC-8_3.9x4.9mm_P1.27mm, F.Cu at (119.4, 107.9)
Other:
- board outline added: 65 x 65 mm

Commit message: layout not routed
Parts:
- moved J5 54.8 mm to (133.4, 137.7), turned to 90 degrees
- moved J6 42.7 mm to (95.3, 107.3), turned to 0 degrees
Changed lines of the file:
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@@
   )
   (footprint "Connector_JST:JST_EH_B2B-EH-A_1x02_P2.50mm_Vertical" (layer "F.Cu")
-    (at 129.606851 132.669987 -90)
+    (at 95.316851 107.269987)
     (descr "JST EH series connector, B2B-EH-A (http://www.jst-mfg.com/product/pdf/eng/eEH.pdf), generated with kicad-footprint-generator")
     (tags "connector JST EH vertical")
@@
     (property "Sheetname" "Battery_protections")
     (attr through_hole)
-    (fp_text reference "J6" (at 1.25 -2.8 90) (layer "F.SilkS")
-      (effects (font (size 1 1) (thickness 0.15)))
-    )
-    (fp_text value "thermistor" (at 1.25 3.4 90) (layer "F.Fab")
-      (effects (font (size 1 1) (thickness 0.15)))
-    )
-    (fp_text user "${REFERENCE}" (at 1.25 1.5 90) (layer "F.Fab")
+    (fp_text reference "J6" (at 1.25 -2.8) (layer "F.SilkS")
+      (effects (font (size 1 1) (thickness 0.15)))
+    )
+    (fp_text value "thermistor" (at 1.25 3.4) (layer "F.Fab")
+      (effects (font (size 1 1) (thickness 0.15)))
+    )
+    (fp_text user "${REFERENCE}" (at 1.25 1.5) (layer "F.Fab")
       (effects (font (size 1 1) (thickness 0.15)))
     )
@@
     (fp_line (start -2.91 0.11) (end -2.91 2.61) (layer "F.Fab") (width 0.1))
     (fp_line (start -2.5 -1.6) (end -2.5 2.2) (layer "F.Fab") (width 0.1))
-    (pad "1" thru_hole roundrect (at 0 0 270) (size 1.7 2) (drill 1) (layers *.Cu *.Mask) (roundrect_rratio 0.147059)
+    (pad "1" thru_hole roundrect (at 0 0) (size 1.7 2) (drill 1) (layers *.Cu *.Mask) (roundrect_rratio 0.147059)
       (net 5 "/12V Boost converter/GND2") (pinfunction "Pin_1") (pintype "passive"))
-    (pad "2" thru_hole oval (at 2.5 0 270) (size 1.7 2) (drill 1) (layers *.Cu *.Mask)
+    (pad "2" thru_hole oval (at 2.5 0) (size 1.7 2) (drill 1) (layers *.Cu *.Mask)
       (net 31 "Net-(J6-Pad2)") (pinfunction "Pin_2") (pintype "passive"))
     (model "${KICAD6_3DMODEL_DIR}/Connector_JST.3dshapes/JST_EH_B2B-EH-A_1x02_P2.50mm_Vertical.wrl"
@@
   )
   (footprint "Connector_JST:JST_EH_B4B-EH-A_1x04_P2.50mm_Vertical" (layer "F.Cu")
-    (at 126.511851 83.409987)
+    (at 133.416851 137.749987 90)
     (descr "JST EH series connector, B4B-EH-A (http://www.jst-mfg.com/product/pdf/eng/eEH.pdf), generated with kicad-footprint-generator")
     (tags "connector JST EH vertical")
@@
     (property "Sheetname" "")
     (attr through_hole)
-    (fp_text reference "J5" (at 3.75 -2.8) (layer "F.SilkS")
-      (effects (font (size 1 1) (thickness 0.15)))
-    )
-    (fp_text value "4pin JST" (at 3.75 3.4) (layer "F.Fab")
-      (effects (font (size 1 1) (thickness 0.15)))
-    )
-    (fp_text user "${REFERENCE}" (at 3.75 1.5) (layer "F.Fab")
+    (fp_text reference "J5" (at 3.75 -2.8 90) (layer "F.SilkS")
+      (effects (font (size 1 1) (thickness 0.15)))
+    )
+    (fp_text value "4pin JST" (at 3.75 3.4 90) (layer "F.Fab")
+      (effects (font (size 1 1) (thickness 0.15)))
+    )
+    (fp_text user "${REFERENCE}" (at 3.75 1.5 90) (layer "F.Fab")
       (effects (font (size 1 1) (thickness 0.15)))
     )
@@
     (fp_line (start 10 -1.6) (end -2.5 -1.6) (layer "F.Fab") (width 0.1))
     (fp_line (start -2.5 2.2) (end 10 2.2) (layer "F.Fab") (width 0.1))
-    (pad "1" thru_hole roundrect (at 0 0) (size 1.7 1.95) (drill 0.95) (layers *.Cu *.Mask) (roundrect_rratio 0.147059)
+    (pad "1" thru_hole roundrect (at 0 0 90) (size 1.7 1.95) (drill 0.95) (layers *.Cu *.Mask) (roundrect_rratio 0.147059)
       (net 26 "/Batt +") (pinfunction "Pin_1") (pintype "passive"))
-    (pad "2" thru_hole oval (at 2.5 0) (size 1.7 1.95) (drill 0.95) (layers *.Cu *.Mask)
+    (pad "2" thru_hole oval (at 2.5 0 90) (size 1.7 1.95) (drill 0.95) (layers *.Cu *.Mask)
       (net 1 "/SW_Batt +") (pinfunction "Pin_2") (pintype "passive"))
-    (pad "3" thru_hole oval (at 5 0) (size 1.7 1.95) (drill 0.95) (layers *.Cu *.Mask)
+    (pad "3" thru_hole oval (at 5 0 90) (size 1.7 1.95) (drill 0.95) (layers *.Cu *.Mask)
       (net 27 "/Bal_batt -") (pinfunction "Pin_3") (pintype "passive"))
-    (pad "4" thru_hole oval (at 7.5 0) (size 1.7 1.95) (drill 0.95) (layers *.Cu *.Mask)
+    (pad "4" thru_hole oval (at 7.5 0 90) (size 1.7 1.95) (drill 0.95) (layers *.Cu *.Mask)
       (net 28 "/Bal_batt +") (pinfunction "Pin_4") (pintype "passive"))
     (model "${KICAD6_3DMODEL_DIR}/Connector_JST.3dshapes/JST_EH_B4B-EH-A_1x04_P2.50mm_Vertical.wrl"

Commit message: First layout done
Parts:
- moved J5 59.7 mm to (109.2, 83.1), turned to 180 degrees
- moved D1 40.8 mm to (148.7, 128.1), turned to 180 degrees
- moved R1 39.3 mm to (148.4, 125.8)
- moved J2 22.9 mm to (133.1, 94.5), turned to 90 degrees
- moved C1 20.1 mm to (96.3, 119.2)
- moved C2 20.1 mm to (96.3, 124.5)
- moved U1 20.1 mm to (101.4, 122.3)
- moved C16 16.7 mm to (118.6, 128.9)
- moved Q7 16.7 mm to (115.3, 119.3)
- moved R22 16.7 mm to (125.4, 128.9)
- moved RV3 16.7 mm to (117.8, 134.6)
- moved C14 16.7 mm to (111.4, 121.9)
- moved C15 16.7 mm to (123.2, 123.8)
- moved C17 16.7 mm to (110.2, 129.5)
- moved C18 16.7 mm to (111.4, 126.3)
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Connections:
- J5 pad 4: /Bal_batt + -> /Batt_+
Routing:
- net /Batt +: track 0.00 -> 59.6 mm
- net /SW_Batt +: track 0.00 -> 31.5 mm
- net /CHG +: track 0.00 -> 16.9 mm
- net /12V: track 0.00 -> 14.7 mm
- net /Battery_protections/VC1_CB: track 0.00 -> 7.03 mm
- net Net-(Q1-Pad1): track 0.00 -> 6.73 mm
- net Net-(D5-Pad1): track 0.00 -> 6.69 mm
- net /Battery_protections/VC1: track 0.00 -> 6.51 mm
- net Net-(C13-Pad1): track 0.00 -> 4.54 mm
- net Net-(Q1-Pad2): track 0.00 -> 4.40 mm
- net GND: track 0.00 -> 4.05 mm
- net Net-(Q2-Pad3): track 0.00 -> 3.81 mm
- net Net-(Q5-Pad3): track 0.00 -> 3.69 mm
- net Net-(Q4-Pad3): track 0.00 -> 3.61 mm
- net Net-(R3-Pad2): track 0.00 -> 3.51 mm
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
Commit message: Re took on project started routing
Parts:
- moved J6 2.27 mm to (109.3, 109.0), turned to 180 degrees
- moved Q8 2.16 mm to (118.7, 114.9)
- moved R18 0.20 mm to (114.2, 114.9)
Routing:
- net /SW_Batt +: track 31.5 -> 59.9 mm
- net /Batt +: track 59.6 -> 65.9 mm
- net Net-(J6-Pad2): track 0.00 -> 5.89 mm
- net /Battery_protections/VC2: track 2.42 -> 5.53 mm
- net Net-(C10-Pad1): track 0.00 -> 2.25 mm
Changed lines of the file:
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@@
   )
   (footprint "Resistor_SMD:R_0805_2012Metric_Pad1.20x1.40mm_HandSolder" (layer "F.Cu")
-    (at 113.985851 114.888336 -90)
+    (at 114.186851 114.879987 -90)
     (descr "Resistor SMD 0805 (2012 Metric), square (rectangular) end terminal, IPC_7351 nominal with elongated pad for handsoldering. (Body size source: IPC-SM-782 page 72, https://www.pcb-3d.com/wordpress/wp-content/uploads/ipc-sm-782a_amendment_1_and_2.pdf), generated with kicad-footprint-generator")
     (tags "resistor handsolder")
@@
   )
   (footprint "Connector_JST:JST_EH_B2B-EH-A_1x02_P2.50mm_Vertical" (layer "F.Cu")
-    (at 107.020851 109.001987)
+    (at 109.286851 109.001987 180)
     (descr "JST EH series connector, B2B-EH-A (http://www.jst-mfg.com/product/pdf/eng/eEH.pdf), generated with kicad-footprint-generator")
     (tags "connector JST EH vertical")
@@
     (fp_line (start -2.91 0.11) (end -2.91 2.61) (layer "F.Fab") (width 0.1))
     (fp_line (start -2.5 -1.6) (end -2.5 2.2) (layer "F.Fab") (width 0.1))
-    (pad "1" thru_hole roundrect (at 0 0) (size 1.7 2) (drill 1) (layers *.Cu *.Mask) (roundrect_rratio 0.147059)
+    (pad "1" thru_hole roundrect (at 0 0 180) (size 1.7 2) (drill 1) (layers *.Cu *.Mask) (roundrect_rratio 0.147059)
       (net 5 "/12V Boost converter/GND2") (pinfunction "Pin_1") (pintype "passive"))
-    (pad "2" thru_hole oval (at 2.5 0) (size 1.7 2) (drill 1) (layers *.Cu *.Mask)
+    (pad "2" thru_hole oval (at 2.5 0 180) (size 1.7 2) (drill 1) (layers *.Cu *.Mask)
       (net 31 "Net-(J6-Pad2)") (pinfunction "Pin_2") (pintype "passive"))
     (model "${KICAD6_3DMODEL_DIR}/Connector_JST.3dshapes/JST_EH_B2B-EH-A_1x02_P2.50mm_Vertical.wrl"
@@
   )
   (footprint "Package_TO_SOT_SMD:SOT-323_SC-70" (layer "F.Cu")
-    (at 116.525851 114.888336 90)
+    (at 118.684851 114.888336 90)
     (descr "SOT-323, SC-70")
     (tags "SOT-323 SC-70")
@@
   (gr_rect (start 72.456851 77.829987) (end 137.456851 142.829987) (layer "Edge.Cuts") (width 0.05) (fill none))
   (segment (start 108.016851 86.314987) (end 113.096851 86.314987) (width 1.1938) (layer "F.Cu") (net 1))
+  (segment (start 75.504851 114.889987) (end 76.647851 114.889987) (width 0.3048) (layer "F.Cu") (net 1))
+  (segment (start 114.200851 113.865987) (end 114.200851 108.538336) (width 0.3048) (layer "F.Cu") (net 1))
+  (segment (start 111.540851 103.967987) (end 111.540851 108.253987) (width 0.3048) (layer "F.Cu") (net 1))
   (segment (start 106.726851 83.125987) (end 106.726851 85.024987) (width 1.1938) (layer "F.Cu") (net 1))
+  (segment (start 74.488851 113.873987) (end 75.504851 114.889987) (width 0.3048) (layer "F.Cu") (net 1))
   (segment (start 114.200851 87.418987) (end 114.200851 108.538336) (width 1.1938) (layer "F.Cu") (net 1))
+  (segment (start 111.826851 108.539987) (end 111.828502 108.538336) (width 0.3048) (layer "F.Cu") (net 1))
+  (segment (start 76.647851 114.889987) (end 76.653851 114.883987) (width 0.3048) (layer "F.Cu") (net 1))
+  (segment (start 111.828502 108.538336) (end 114.200851 108.538336) (width 0.3048) (layer "F.Cu") (net 1))
+  (segment (start 75.208851 101.469987) (end 74.488851 102.189987) (width 0.3048) (layer "F.Cu") (net 1))
+  (segment (start 74.488851 102.189987) (end 74.488851 113.873987) (width 0.3048) (layer "F.Cu") (net 1))
   (segment (start 113.096851 86.314987) (end 114.200851 87.418987) (width 1.1938) (layer "F.Cu") (net 1))
+  (segment (start 111.540851 108.253987) (end 111.826851 108.539987) (width 0.3048) (layer "F.Cu") (net 1))
+  (segment (start 114.186851 113.879987) (end 114.200851 113.865987) (width 0.3048) (layer "F.Cu") (net 1))
   (segment (start 106.726851 85.024987) (end 108.016851 86.314987) (width 1.1938) (layer "F.Cu") (net 1))
+  (segment (start 75.891851 101.469987) (end 75.208851 101.469987) (width 0.3048) (layer "F.Cu") (net 1))
   (segment (start 124.591851 79.964987) (end 127.456851 82.829987) (width 1.1938) (layer "F.Cu") (net 2))
   (segment (start 133.6592 99.707638) (end 133.716851 99.649987) (width 0.508) (layer "F.Cu") (net 5))
@@
   (segment (start 78.150351 95.056487) (end 77.028851 95.056487) (width 0.3048) (layer "F.Cu") (net 8))
   (segment (start 80.129351 95.922987) (end 79.016851 95.922987) (width 0.3048) (layer "F.Cu") (net 8))
+  (segment (start 77.32185 108.500988) (end 77.964852 108.500988) (width 0.3048) (layer "F.Cu") (net 9))
   (segment (start 76.653851 110.857487) (end 76.378351 110.581987) (width 0.3048) (layer "F.Cu") (net 9))
+  (segment (start 77.028851 108.793987) (end 77.32185 108.500988) (width 0.3048) (layer "F.Cu") (net 9))
+  (segment (start 77.028851 109.931487) (end 77.028851 108.793987) (width 0.3048) (layer "F.Cu") (net 9))
   (segment (start 76.653851 112.883987) (end 76.653851 110.857487) (width 0.3048) (layer "F.Cu") (net 9))
+  (segment (start 76.378351 110.581987) (end 77.028851 109.931487) (width 0.3048) (layer "F.Cu") (net 9))
   (segment (start 78.61485 108.500988) (end 78.61485 110.420488) (width 0.3048) (layer "F.Cu") (net 10))
   (segment (start 78.425851 111.714987) (end 78.425851 110.609487) (width 0.3048) (layer "F.Cu") (net 10))
@@
   (segment (start 79.264852 108.997988) (end 79.695851 109.428987) (width 0.3048) (layer "F.Cu") (net 11))
   (segment (start 82.263351 109.964487) (end 82.263351 110.581987) (width 0.3048) (layer "F.Cu") (net 11))
+  (segment (start 81.956351 108.031987) (end 81.966351 108.041987) (width 0.3048) (layer "F.Cu") (net 12))
+  (segment (start 79.91485 108.500988) (end 80.62385 108.500988) (width 0.3048) (layer "F.Cu") (net 12))
+  (segment (start 80.62385 108.500988) (end 81.092851 108.031987) (width 0.3048) (layer "F.Cu") (net 12))
+  (segment (start 81.092851 108.031987) (end 81.956351 108.031987) (width 0.3048) (layer "F.Cu") (net 12))
   (segment (start 127.9542 103.207638) (end 128.971851 102.189987) (width 1.1938) (layer "F.Cu") (net 22))
   (segment (start 128.971851 102.189987) (end 133.716851 102.189987) (width 1.1938) (layer "F.Cu") (net 22))
@@
   (segment (start 84.354351 96.572987) (end 83.222851 96.572987) (width 0.3048) (layer "F.Cu") (net 24))
   (segment (start 119.700851 108.538336) (end 121.900851 108.538336) (width 1.1938) (layer "F.Cu") (net 25))
+  (segment (start 78.947851 97.222987) (end 78.552851 97.617987) (width 0.3048) (layer "F.Cu") (net 26))
   (segment (start 95.570851 81.234987) (end 107.335851 81.234987) (width 0.3048) (layer "F.Cu") (net 26))
   (segment (start 89.601851 87.203987) (end 95.570851 81.234987) (width 0.3048) (layer "F.Cu") (net 26))
   (segment (start 109.522851 82.829987) (end 121.956851 82.829987) (width 1.1938) (layer "F.Cu") (net 26))
+  (segment (start 79.610851 100.199987) (end 81.241851 100.199987) (width 0.3048) (layer "F.Cu") (net 26))
   (segment (start 89.601851 100.030987) (end 89.601851 87.203987) (width 0.3048) (layer "F.Cu") (net 26))
   (segment (start 81.981851 102.316987) (end 87.315851 102.316987) (width 0.3048) (layer "F.Cu") (net 26))
@@
   (segment (start 87.315851 102.316987) (end 89.601851 100.030987) (width 0.3048) (layer "F.Cu") (net 26))
   (segment (start 81.241851 100.199987) (end 81.241851 101.576987) (width 0.3048) (layer "F.Cu") (net 26))
+  (segment (start 80.129351 97.222987) (end 78.947851 97.222987) (width 0.3048) (layer "F.Cu") (net 26))
+  (segment (start 78.552851 97.617987) (end 78.552851 99.141987) (width 0.3048) (layer "F.Cu") (net 26))
+  (segment (start 78.552851 99.141987) (end 79.610851 100.199987) (width 0.3048) (layer "F.Cu") (net 26))
+  (segment (start 106.786851 109.001987) (end 102.652851 109.001987) (width 0.3048) (layer "F.Cu") (net 31))
+  (segment (start 102.652851 109.001987) (end 101.412851 107.761987) (width 0.3048) (layer "F.Cu") (net 31))
   (segment (start 84.354351 97.872987) (end 86.534851 97.872987) (width 0.3048) (layer "F.Cu") (net 32))
   (segment (start 86.534851 97.872987) (end 87.321851 98.659987) (width 0.3048) (layer "F.Cu") (net 32))

Commit message: Added gitignore for backup file tracking
Routing:
- net (no net): track 0.00 -> 3.87 mm
Changed lines of the file:
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@@
   )
   (gr_rect (start 72.456851 77.829987) (end 137.456851 142.829987) (layer "Edge.Cuts") (width 0.05) (fill none))
+  (segment (start 86.426851 105.745987) (end 85.664851 104.983987) (width 0.3048) (layer "F.Cu") (net 0))
+  (segment (start 89.220851 105.745987) (end 86.426851 105.745987) (width 0.3048) (layer "F.Cu") (net 0))
   (segment (start 108.016851 86.314987) (end 113.096851 86.314987) (width 1.1938) (layer "F.Cu") (net 1))
   (segment (start 75.504851 114.889987) (end 76.647851 114.889987) (width 0.3048) (layer "F.Cu") (net 1))
