File: Ki_PCB.kicad_sch (KiCad schematic)
At the start: 9 parts, among them J1 0039301020, J2 B3B-XH-AM(LF)(SN), J3 0039301020, J4 0470531000, J5 4pin JST, SW1 SW_Push

Commit message: Fixes brought on laptop
Parts:
- D2: footprint (none) -> LED_THT:LED_D3.0mm
- SW1: footprint (none) -> laptop_Library:SW_Header_toggle_switch
Connections:
- net Batt +: now also SW1.1
- net SW_Batt +: now also SW1.2
- no-connect marks 3 -> 1
Other:
- sheet PWM_generation ports: added SW_Batt +; removed Batt +
- note removed: "footprint to be added: switch"
- moved on the sheet: D2
Changed lines of the file:
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@@
   )
   (no_connect (at 187.96 41.91))
-  (no_connect (at 191.77 104.14))
-  (no_connect (at 181.61 104.14))
   (wire (pts (xy 175.26 44.45) (xy 187.96 44.45))
     (stroke (width 0) (type default) (color 0 0 0 0))
@@
     (stroke (width 0) (type default) (color 0 0 0 0))
   )
-  (wire (pts (xy 168.91 118.11) (xy 181.61 118.11))
+  (wire (pts (xy 170.18 118.11) (xy 182.88 118.11))
     (stroke (width 0) (type default) (color 0 0 0 0))
   )
@@
     (stroke (width 0) (type default) (color 0 0 0 0))
   )
+  (wire (pts (xy 170.18 104.14) (xy 181.61 104.14))
+    (stroke (width 0) (type default) (color 0 0 0 0))
+  )
   (wire (pts (xy 30.48 115.57) (xy 43.18 115.57))
     (stroke (width 0) (type default) (color 0 0 0 0))
@@
     (stroke (width 0) (type default) (color 0 0 0 0))
   )
-  (wire (pts (xy 69.85 33.02) (xy 80.01 33.02))
+  (wire (pts (xy 68.58 33.02) (xy 80.01 33.02))
     (stroke (width 0) (type default) (color 0 0 0 0))
   )
@@
     (stroke (width 0) (type default) (color 0 0 0 0))
   )
+  (wire (pts (xy 191.77 104.14) (xy 203.2 104.14))
+    (stroke (width 0) (type default) (color 0 0 0 0))
+  )
   (wire (pts (xy 120.65 29.21) (xy 146.05 29.21))
     (stroke (width 0) (type default) (color 0 0 0 0))
@@
     (stroke (width 0) (type default) (color 0 0 0 0))
   )
-  (wire (pts (xy 189.23 118.11) (xy 201.93 118.11))
+  (wire (pts (xy 190.5 118.11) (xy 203.2 118.11))
     (stroke (width 0) (type default) (color 0 0 0 0))
   )
@@
     (effects (font (size 1.27 1.27)) (justify left bottom))
   )
-  (text "footprint to be added:\nswitch\n\n" (at 46.99 71.12 0)
-    (effects (font (size 1.27 1.27)) (justify left bottom))
-  )
-  (text "charge level indicator\n" (at 176.53 123.19 0)
+  (text "charge level indicator\n" (at 177.8 123.19 0)
     (effects (font (size 1.27 1.27)) (justify left bottom))
   )
@@
     (effects (font (size 1.27 1.27)) (justify left bottom))
   )
-  (label "Batt +" (at 69.85 33.02 0)
-    (effects (font (size 1.27 1.27)) (justify left bottom))
-  )
   (label "Bal_batt -" (at 179.07 73.66 0)
     (effects (font (size 1.27 1.27)) (justify left bottom))
@@
     (effects (font (size 1.27 1.27)) (justify right bottom))
   )
-  (label "Bal_batt -" (at 201.93 118.11 180)
-    (effects (font (size 1.27 1.27)) (justify right bottom))
+  (label "SW_Batt +" (at 203.2 104.14 180)
+    (effects (font (size 1.27 1.27)) (justify right bottom))
+  )
+  (label "Bal_batt -" (at 203.2 118.11 180)
+    (effects (font (size 1.27 1.27)) (justify right bottom))
+  )
+  (label "SW_Batt +" (at 68.58 33.02 0)
+    (effects (font (size 1.27 1.27)) (justify left bottom))
   )
   (label "Bal_batt +" (at 179.07 71.12 0)
     (effects (font (size 1.27 1.27)) (justify left bottom))
   )
+  (label "Batt +" (at 170.18 104.14 0)
+    (effects (font (size 1.27 1.27)) (justify left bottom))
+  )
   (label "CHG +" (at 43.18 49.53 180)
     (effects (font (size 1.27 1.27)) (justify right bottom))
   )
-  (label "SW_Batt +" (at 63.5 74.93 180)
-    (effects (font (size 1.27 1.27)) (justify right bottom))
+  (label "SW_Batt +" (at 45.72 74.93 0)
+    (effects (font (size 1.27 1.27)) (justify left bottom))
   )
   (label "Batt +" (at 35.56 74.93 180)
@@
     (effects (font (size 1.27 1.27)) (justify right bottom))
   )
-  (label "Bal_batt +" (at 168.91 118.11 0)
+  (label "Bal_batt +" (at 170.18 118.11 0)
     (effects (font (size 1.27 1.27)) (justify left bottom))
   )
@@
     (pin "2")
   )
-  (symbol (lib_id "Device:LED") (at 185.42 118.11 180) (unit 1)
+  (symbol (lib_id "Device:LED") (at 186.69 118.11 180) (unit 1)
     (in_bom no) (on_board no) (fields_autoplaced)
-    (property "Reference" "D2" (id 0) (at 187.0075 110.49 0))
-    (property "Value" "LED" (id 1) (at 187.0075 113.03 0))
-    (property "Footprint" "" (id 2) (at 185.42 118.11 0)
-      (effects (font (size 1.27 1.27)) hide)
-    )
-    (property "Datasheet" "~" (id 3) (at 185.42 118.11 0)
+    (property "Reference" "D2" (id 0) (at 188.2775 110.49 0))
+    (property "Value" "LED" (id 1) (at 188.2775 113.03 0))
+    (property "Footprint" "LED_THT:LED_D3.0mm" (id 2) (at 186.69 118.11 0)
+      (effects (font (size 1.27 1.27)) hide)
+    )
+    (property "Datasheet" "~" (id 3) (at 186.69 118.11 0)
       (effects (font (size 1.27 1.27)) hide)
     )
@@
     (property "Reference" "SW1" (id 0) (at 186.69 96.52 0))
     (property "Value" "SW_Push" (id 1) (at 186.69 99.06 0))
-    (property "Footprint" "" (id 2) (at 186.69 99.06 0)
+    (property "Footprint" "laptop_Library:SW_Header_toggle_switch" (id 2) (at 186.69 99.06 0)
       (effects (font (size 1.27 1.27)) hide)
     )
@@
       (effects (font (size 1.27 1.27)) (justify right))
     )
-    (pin "Batt +" input (at 80.01 33.02 180)
+    (pin "SW_Batt +" input (at 80.01 33.02 180)
       (effects (font (size 1.27 1.27)) (justify left))
     )
@@
     )
     (path "/1fffe7b2-290f-4d56-a315-c92fd31a7edf"
-      (reference "D2") (unit 1) (value "LED") (footprint "")
+      (reference "D2") (unit 1) (value "LED") (footprint "LED_THT:LED_D3.0mm")
     )
     (path "/9ab53ca4-c94c-4c0f-9710-20b56a11033f/f3fe62bc-01bc-4418-80b6-e3e4e80767cf"
@@
       (reference "R13") (unit 1) (value "100") (footprint "Resistor_SMD:R_0805_2012Metric_Pad1.20x1.40mm_HandSolder")
     )
-    (path "/a43c876c-93ca-4457-bd54-0a8c2951e964/9756f229-7068-4cb7-8d79-ddbc98c7403d"
-      (reference "R14") (unit 1) (value "10K") (footprint "Resistor_SMD:R_0805_2012Metric_Pad1.20x1.40mm_HandSolder")
-    )
     (path "/58f11461-4943-4ae3-b4d8-49e23e57c963/a34352e0-3585-4f98-8f96-4534b54b2b61"
       (reference "R15") (unit 1) (value "113K") (footprint "Resistor_SMD:R_0805_2012Metric_Pad1.20x1.40mm_HandSolder")
@@
     )
     (path "/2f86d018-8b99-49dd-95b5-376a07db1ce2"
-      (reference "SW1") (unit 1) (value "SW_Push") (footprint "")
+      (reference "SW1") (unit 1) (value "SW_Push") (footprint "laptop_Library:SW_Header_toggle_switch")
     )
     (path "/d0cbe6c3-ddca-405e-bd7e-804b30aab2db/3b288e81-687d-40b3-bfb0-8cbd4c5e3dd2"

Commit message: First layout done
Other:
- sheet Battery_protections ports: added Bal_batt_+, Bal_batt_-; removed none
Changed lines of the file:
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@@
     (stroke (width 0) (type default) (color 0 0 0 0))
   )
-  (wire (pts (xy 30.48 110.49) (xy 43.18 110.49))
+  (wire (pts (xy 30.48 110.49) (xy 63.5 110.49))
     (stroke (width 0) (type default) (color 0 0 0 0))
   )
@@
     (stroke (width 0) (type default) (color 0 0 0 0))
   )
+  (wire (pts (xy 68.58 115.57) (xy 68.58 105.41))
+    (stroke (width 0) (type default) (color 0 0 0 0))
+  )
   (wire (pts (xy 170.18 118.11) (xy 182.88 118.11))
     (stroke (width 0) (type default) (color 0 0 0 0))
@@
     (stroke (width 0) (type default) (color 0 0 0 0))
   )
-  (wire (pts (xy 30.48 115.57) (xy 43.18 115.57))
+  (wire (pts (xy 30.48 115.57) (xy 68.58 115.57))
     (stroke (width 0) (type default) (color 0 0 0 0))
   )
@@
     (stroke (width 0) (type default) (color 0 0 0 0))
   )
-  (wire (pts (xy 67.31 100.33) (xy 77.47 100.33))
-    (stroke (width 0) (type default) (color 0 0 0 0))
-  )
-  (wire (pts (xy 66.04 97.79) (xy 77.47 97.79))
+  (wire (pts (xy 67.31 97.79) (xy 77.47 97.79))
     (stroke (width 0) (type default) (color 0 0 0 0))
   )
@@
     (stroke (width 0) (type default) (color 0 0 0 0))
   )
-  (wire (pts (xy 66.04 113.03) (xy 66.04 97.79))
-    (stroke (width 0) (type default) (color 0 0 0 0))
-  )
   (wire (pts (xy 113.03 54.61) (xy 129.54 54.61))
     (stroke (width 0) (type default) (color 0 0 0 0))
@@
     (stroke (width 0) (type default) (color 0 0 0 0))
   )
+  (wire (pts (xy 77.47 100.33) (xy 63.5 100.33))
+    (stroke (width 0) (type default) (color 0 0 0 0))
+  )
   (wire (pts (xy 60.96 74.93) (xy 60.96 77.47))
     (stroke (width 0) (type default) (color 0 0 0 0))
@@
     (stroke (width 0) (type default) (color 0 0 0 0))
   )
+  (wire (pts (xy 66.04 102.87) (xy 66.04 113.03))
+    (stroke (width 0) (type default) (color 0 0 0 0))
+  )
   (wire (pts (xy 45.72 74.93) (xy 60.96 74.93))
     (stroke (width 0) (type default) (color 0 0 0 0))
@@
     (stroke (width 0) (type default) (color 0 0 0 0))
   )
+  (wire (pts (xy 63.5 100.33) (xy 63.5 110.49))
+    (stroke (width 0) (type default) (color 0 0 0 0))
+  )
   (wire (pts (xy 43.18 52.07) (xy 43.18 55.88))
     (stroke (width 0) (type default) (color 0 0 0 0))
@@
     (stroke (width 0) (type default) (color 0 0 0 0))
   )
+  (wire (pts (xy 68.58 105.41) (xy 77.47 105.41))
+    (stroke (width 0) (type default) (color 0 0 0 0))
+  )
   (wire (pts (xy 35.56 49.53) (xy 71.12 49.53))
     (stroke (width 0) (type default) (color 0 0 0 0))
@@
     (stroke (width 0) (type default) (color 0 0 0 0))
   )
+  (wire (pts (xy 77.47 102.87) (xy 66.04 102.87))
+    (stroke (width 0) (type default) (color 0 0 0 0))
+  )
   (wire (pts (xy 179.07 78.74) (xy 190.5 78.74))
     (stroke (width 0) (type default) (color 0 0 0 0))
@@
     (effects (font (size 1.27 1.27)) (justify left bottom))
   )
-  (label "Batt -" (at 67.31 100.33 0)
+  (label "Batt -" (at 67.31 97.79 0)
     (effects (font (size 1.27 1.27)) (justify left bottom))
   )
@@
       (effects (font (size 1.27 1.27)) (justify left))
     )
-    (pin "batt -" input (at 77.47 100.33 180)
-      (effects (font (size 1.27 1.27)) (justify left))
-    )
-    (pin "Batt mid" input (at 77.47 97.79 180)
+    (pin "batt -" input (at 77.47 97.79 180)
+      (effects (font (size 1.27 1.27)) (justify left))
+    )
+    (pin "Batt mid" input (at 77.47 102.87 180)
       (effects (font (size 1.27 1.27)) (justify left))
     )
@@
       (effects (font (size 1.27 1.27)) (justify right))
     )
-  )
+    (pin "Bal_batt_+" input (at 77.47 100.33 180)
+      (effects (font (size 1.27 1.27)) (justify left))
+    )
+    (pin "Bal_batt_-" input (at 77.47 105.41 180)
+      (effects (font (size 1.27 1.27)) (justify left))
+    )
+  )
