File: PWM_generation.kicad_sch (KiCad schematic)
At the start: 9 parts, among them U1 LDL1117S50R, U2 TLC555CPWR

Commit message: Fixes brought on laptop
Connections:
- net Batt + renamed SW_Batt +
Changed lines of the file:
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@@
     (effects (font (size 1.27 1.27)) (justify left bottom))
   )
-  (label "Batt +" (at 29.21 36.83 0)
+  (label "SW_Batt +" (at 29.21 36.83 0)
     (effects (font (size 1.27 1.27)) (justify left bottom))
   )
-  (hierarchical_label "Batt +" (shape input) (at 29.21 36.83 180)
+  (hierarchical_label "SW_Batt +" (shape input) (at 29.21 36.83 180)
     (effects (font (size 1.27 1.27)) (justify right))
   )

Commit message: 1st Gerber creatd  Please enter the commit message for your changes. Lines starting
Connections:
- net at R2.2, U2.12 (DIS): now also RV1.1; no longer RV1.3
- net at C3.1, RV1.2, U2.10 (THR)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: now also RV1.3; no longer RV1.1
Changed lines of the file:
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@@
   (symbol (lib_id "Device:R_Potentiometer_US") (at 123.19 90.17 0) (mirror x) (unit 1)
     (in_bom yes) (on_board yes) (fields_autoplaced)
-    (property "Reference" "RV1" (id 0) (at 120.65 88.8999 0)
+    (property "Reference" "RV1" (id 0) (at 120.65 91.4401 0)
       (effects (font (size 1.27 1.27)) (justify right))
     )
-    (property "Value" "22K" (id 1) (at 120.65 91.4399 0)
+    (property "Value" "22K" (id 1) (at 120.65 88.9001 0)
       (effects (font (size 1.27 1.27)) (justify right))
     )
@@
       (effects (font (size 1.27 1.27)) hide)
     )
-    (property "Part number" "PC16SH-10IP06-223A2020-TA" (id 4) (at 123.19 90.17 90)
+    (property "Part number" "PC16SH-10IP06-223A2020-TA" (id 4) (at 132.08 88.9 90)
       (effects (font (size 1.27 1.27)) hide)
     )
-    (property "Digikey link" "https://www.digikey.ca/en/products/detail/amphenol-piher-sensing-systems/PC16SH-10IP06-223A2020-TA/16028525?s=N4IgTCBcDaIIwE4EGYC0AFAwnAbAZQAlU4AGASXRJ1TDGQEEwSnUAVe1AOQBEQBdAL5A" (id 5) (at 123.19 90.17 90)
+    (property "Digikey link" "https://www.digikey.ca/en/products/detail/amphenol-piher-sensing-systems/PC16SH-10IP06-223A2020-TA/16028525?s=N4IgTCBcDaIIwE4EGYC0AFAwnAbAZQAlU4AGASXRJ1TDGQEEwSnUAVe1AOQBEQBdAL5A" (id 5) (at 114.3 90.17 90)
       (effects (font (size 1.27 1.27)) hide)
     )
