File: boost_converter.kicad_sch (KiCad schematic)
At the start: 21 parts, among them Q7 SI2102A-TP, Q8 SI2102A-TP, U8 TL5001CDR

Commit message: 1st Gerber creatd  Please enter the commit message for your changes. Lines starting
Parts:
- renumbered C14 to C15, C15 to C16, C16 to C17, C17 to C18, C18 to C19, C19 to C20, C20 to C21, D6 to D4, R15 to R14, R16 to R15, R17 to R16, R18 to R17, R19 to R18, R20 to R19, R21 to R20, R22 to R21
Connections:
- net GND2: now also Q7.2 (S), Q8.2 (S); no longer Q7.3 (D), Q8.3 (D)
- net at Q8.1 (G), R18.2: now also Q7.3 (D); no longer Q7.2 (S)
- net at D4.2 (A), L1.2: now also Q8.3 (D); no longer Q8.2 (S)
Changed lines of the file:
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@@
   (symbol (lib_id "Device:R_US") (at 82.55 88.9 180) (unit 1)
     (in_bom yes) (on_board yes)
-    (property "Reference" "R16" (id 0) (at 83.82 85.09 90))
+    (property "Reference" "R15" (id 0) (at 83.82 85.09 90))
     (property "Value" "100K" (id 1) (at 83.82 92.71 90))
     (property "Footprint" "Resistor_SMD:R_0805_2012Metric_Pad1.20x1.40mm_HandSolder" (id 2) (at 81.534 88.646 90)
@@
   (symbol (lib_id "Device:C_Polarized_Small_US") (at 208.28 62.23 0) (unit 1)
     (in_bom yes) (on_board yes) (fields_autoplaced)
-    (property "Reference" "C20" (id 0) (at 210.82 60.5281 0)
+    (property "Reference" "C21" (id 0) (at 210.82 60.5281 0)
       (effects (font (size 1.27 1.27)) (justify left))
     )
@@
   (symbol (lib_id "Device:R_US") (at 139.7 60.96 0) (unit 1)
     (in_bom yes) (on_board yes)
-    (property "Reference" "R19" (id 0) (at 138.43 66.04 90))
+    (property "Reference" "R18" (id 0) (at 138.43 66.04 90))
     (property "Value" "10K" (id 1) (at 138.43 55.88 90))
     (property "Footprint" "Resistor_SMD:R_0805_2012Metric_Pad1.20x1.40mm_HandSolder" (id 2) (at 140.716 61.214 90)
@@
   (symbol (lib_id "Device:R_US") (at 189.23 90.17 0) (mirror y) (unit 1)
     (in_bom yes) (on_board yes)
-    (property "Reference" "R21" (id 0) (at 190.5 93.98 90))
+    (property "Reference" "R20" (id 0) (at 190.5 93.98 90))
     (property "Value" "2K7" (id 1) (at 190.5 86.36 90))
     (property "Footprint" "Resistor_SMD:R_0805_2012Metric_Pad1.20x1.40mm_HandSolder" (id 2) (at 188.214 90.424 90)
@@
   (symbol (lib_id "Device:R_US") (at 125.73 64.77 0) (unit 1)
     (in_bom yes) (on_board yes)
-    (property "Reference" "R18" (id 0) (at 124.46 69.85 90))
+    (property "Reference" "R17" (id 0) (at 124.46 69.85 90))
     (property "Value" "10K" (id 1) (at 124.46 59.69 90))
     (property "Footprint" "Resistor_SMD:R_0805_2012Metric_Pad1.20x1.40mm_HandSolder" (id 2) (at 126.746 65.024 90)
@@
   (symbol (lib_id "Device:C") (at 128.27 86.36 180) (unit 1)
     (in_bom yes) (on_board yes) (fields_autoplaced)
-    (property "Reference" "C18" (id 0) (at 132.08 85.0899 0)
+    (property "Reference" "C19" (id 0) (at 132.08 85.0899 0)
       (effects (font (size 1.27 1.27)) (justify right))
     )
@@
   (symbol (lib_id "Device:C") (at 119.38 92.71 180) (unit 1)
     (in_bom yes) (on_board yes) (fields_autoplaced)
-    (property "Reference" "C17" (id 0) (at 123.19 91.4399 0)
+    (property "Reference" "C18" (id 0) (at 123.19 91.4399 0)
       (effects (font (size 1.27 1.27)) (justify right))
     )
@@
   (symbol (lib_id "Device:C") (at 77.47 72.39 270) (mirror x) (unit 1)
     (in_bom yes) (on_board yes) (fields_autoplaced)
-    (property "Reference" "C16" (id 0) (at 77.47 64.77 90))
+    (property "Reference" "C17" (id 0) (at 77.47 64.77 90))
     (property "Value" "1uF" (id 1) (at 77.47 67.31 90))
     (property "Footprint" "Capacitor_SMD:C_0805_2012Metric_Pad1.18x1.45mm_HandSolder" (id 2) (at 73.66 71.4248 0)
@@
   (symbol (lib_id "Device:R_US") (at 74.93 88.9 180) (unit 1)
     (in_bom yes) (on_board yes)
-    (property "Reference" "R15" (id 0) (at 76.2 85.09 90))
+    (property "Reference" "R14" (id 0) (at 76.2 85.09 90))
     (property "Value" "113K" (id 1) (at 76.2 92.71 90))
     (property "Footprint" "Resistor_SMD:R_0805_2012Metric_Pad1.20x1.40mm_HandSolder" (id 2) (at 73.914 88.646 90)
@@
   (symbol (lib_id "Device:R_US") (at 198.12 68.58 0) (mirror y) (unit 1)
     (in_bom yes) (on_board yes)
-    (property "Reference" "R22" (id 0) (at 199.39 72.39 90))
+    (property "Reference" "R21" (id 0) (at 199.39 72.39 90))
     (property "Value" "200R" (id 1) (at 199.39 64.77 90))
     (property "Footprint" "Resistor_SMD:R_0805_2012Metric_Pad1.20x1.40mm_HandSolder" (id 2) (at 197.104 68.834 90)
@@
     (pin "2")
   )
-  (symbol (lib_id "Transistor_FET:SI2102A-TP") (at 157.48 66.04 0) (mirror x) (unit 1)
-    (in_bom yes) (on_board yes)
-    (property "Reference" "Q8" (id 0) (at 163.83 64.7699 0)
-      (effects (font (size 1.27 1.27)) (justify left))
-    )
-    (property "Value" "SI2102A-TP" (id 1) (at 163.83 67.31 0)
-      (effects (font (size 1.27 1.27)) (justify left))
-    )
-    (property "Footprint" "Package_TO_SOT_SMD:SOT-323_SC-70" (id 2) (at 157.48 50.8 0)
+  (symbol (lib_id "Transistor_FET:SI2102A-TP") (at 157.48 66.04 0) (unit 1)
+    (in_bom yes) (on_board yes)
+    (property "Reference" "Q8" (id 0) (at 163.83 67.3101 0)
+      (effects (font (size 1.27 1.27)) (justify left))
+    )
+    (property "Value" "SI2102A-TP" (id 1) (at 163.83 64.77 0)
+      (effects (font (size 1.27 1.27)) (justify left))
+    )
+    (property "Footprint" "Package_TO_SOT_SMD:SOT-323_SC-70" (id 2) (at 157.48 81.28 0)
       (effects (font (size 1.27 1.27) italic) (justify left) hide)
     )
-    (property "Datasheet" "https://www.mccsemi.com/pdf/Products/SI2102A(SOT-323).pdf" (id 3) (at 152.4 48.26 0)
+    (property "Datasheet" "https://www.mccsemi.com/pdf/Products/SI2102A(SOT-323).pdf" (id 3) (at 152.4 83.82 0)
       (effects (font (size 1.27 1.27)) (justify left) hide)
     )
@@
   (symbol (lib_id "Device:R_US") (at 189.23 67.31 0) (mirror y) (unit 1)
     (in_bom yes) (on_board yes)
-    (property "Reference" "R20" (id 0) (at 190.5 71.12 90))
+    (property "Reference" "R19" (id 0) (at 190.5 71.12 90))
     (property "Value" "27K" (id 1) (at 190.5 63.5 90))
     (property "Footprint" "Resistor_SMD:R_0805_2012Metric_Pad1.20x1.40mm_HandSolder" (id 2) (at 188.214 67.564 90)
@@
   (symbol (lib_id "Device:C") (at 66.04 60.96 0) (mirror x) (unit 1)
     (in_bom yes) (on_board yes) (fields_autoplaced)
-    (property "Reference" "C14" (id 0) (at 62.23 59.6899 0)
+    (property "Reference" "C15" (id 0) (at 62.23 59.6899 0)
       (effects (font (size 1.27 1.27)) (justify right))
     )
@@
   (symbol (lib_id "Device:R_US") (at 119.38 82.55 180) (unit 1)
     (in_bom yes) (on_board yes)
-    (property "Reference" "R17" (id 0) (at 120.65 78.74 90))
+    (property "Reference" "R16" (id 0) (at 120.65 78.74 90))
     (property "Value" "12K" (id 1) (at 120.65 86.36 90))
     (property "Footprint" "Resistor_SMD:R_0805_2012Metric_Pad1.20x1.40mm_HandSolder" (id 2) (at 118.364 82.296 90)
@@
   (symbol (lib_id "Device:C") (at 198.12 78.74 180) (unit 1)
     (in_bom yes) (on_board yes)
-    (property "Reference" "C19" (id 0) (at 201.93 77.47 0)
+    (property "Reference" "C20" (id 0) (at 201.93 77.47 0)
       (effects (font (size 1.27 1.27)) (justify right))
     )
@@
   (symbol (lib_id "Device:C") (at 67.31 88.9 0) (mirror x) (unit 1)
     (in_bom yes) (on_board yes) (fields_autoplaced)
-    (property "Reference" "C15" (id 0) (at 63.5 87.6299 0)
+    (property "Reference" "C16" (id 0) (at 63.5 87.6299 0)
       (effects (font (size 1.27 1.27)) (justify right))
     )
@@
   (symbol (lib_id "Device:D_Schottky") (at 170.18 55.88 180) (unit 1)
     (in_bom yes) (on_board yes) (fields_autoplaced)
-    (property "Reference" "D6" (id 0) (at 170.4975 49.53 0))
+    (property "Reference" "D4" (id 0) (at 170.4975 49.53 0))
     (property "Value" "CRS05(TE85L,Q,M)" (id 1) (at 170.4975 52.07 0)
       (effects (font (size 1.27 1.27)) hide)
@@
     (pin "2")
   )
-  (symbol (lib_id "Transistor_FET:SI2102A-TP") (at 137.16 72.39 0) (mirror x) (unit 1)
-    (in_bom yes) (on_board yes)
-    (property "Reference" "Q7" (id 0) (at 143.51 71.1199 0)
-      (effects (font (size 1.27 1.27)) (justify left))
-    )
-    (property "Value" "SI2102A-TP" (id 1) (at 143.51 73.66 0)
-      (effects (font (size 1.27 1.27)) (justify left))
-    )
-    (property "Footprint" "Package_TO_SOT_SMD:SOT-323_SC-70" (id 2) (at 137.16 57.15 0)
+  (symbol (lib_id "Transistor_FET:SI2102A-TP") (at 137.16 72.39 0) (unit 1)
+    (in_bom yes) (on_board yes)
+    (property "Reference" "Q7" (id 0) (at 143.51 73.6601 0)
+      (effects (font (size 1.27 1.27)) (justify left))
+    )
+    (property "Value" "SI2102A-TP" (id 1) (at 143.51 71.12 0)
+      (effects (font (size 1.27 1.27)) (justify left))
+    )
+    (property "Footprint" "Package_TO_SOT_SMD:SOT-323_SC-70" (id 2) (at 137.16 87.63 0)
       (effects (font (size 1.27 1.27) italic) (justify left) hide)
     )
-    (property "Datasheet" "https://www.mccsemi.com/pdf/Products/SI2102A(SOT-323).pdf" (id 3) (at 132.08 54.61 0)
+    (property "Datasheet" "https://www.mccsemi.com/pdf/Products/SI2102A(SOT-323).pdf" (id 3) (at 132.08 90.17 0)
       (effects (font (size 1.27 1.27)) (justify left) hide)
     )
